File: eagle/rpi-pwrbtn.sch (EAGLE design)
At the start: 16 parts, among them IC1 ATTINY85-20SU, IC2 +3V3, X1 ALTPWR

Commit message: Update through-hole schematic and board files.
Parts:
- removed JP1: BTN, jumper:JP1E
- removed JP2: LED, jumper:JP1E
- removed R4: 10k, resistor:R-US_R0603
- removed SV1: RPI, con-lsta:FE13-2
- removed SV2: ICSP, con-lstb:MA03-2
- removed X1: ALTPWR, con-ptr500:AK300/2
- added C3: 100nF, resistor:C-US050-024X044
- added ICSP: (no value), pinhead:PINHD-2X3
- added LED1: STATUS, led:LED3MM
- added R5: 6k2, resistor:R-EU_0204/7
- added R6: 62k, resistor:R-EU_0204/7
- added RESET-B: RESET, switch-omron:10-XX
- added RPI: (no value), pinhead:PINHD-2X13
- added T1: 2N2222, transistor:2N2222
- added VCC: (no value), jumper:SJ
- C1: value 0.1µF -> 100nF; device resistor:C-USC0603K -> resistor:C-US050-024X044
- C2: device resistor:C-USC0603K -> resistor:C-US050-024X044
- IC1: value ATTINY85-20SU -> LD117AV33; device gamaral:TINY85S -> v-reg:LD117AV33
- IC2: value +3V3 -> TINY85P; device linear:MC33269ST-3.3T3 -> gamaral:TINY85P
- J1: device con-jack:JACK-PLUG1 -> con-jack:DCJ0303
- Q1: value (none) -> TIP125; device transistor-power:PMOSFET_PTO220BH -> transistor-power:TIP125
- R1: device resistor:R-US_R0603 -> resistor:R-EU_0204/7
- R2: value 10k -> 330R; device resistor:R-US_R0603 -> resistor:R-EU_0204/7
- R3: value 10k -> 240k; device resistor:R-US_R0603 -> resistor:R-EU_0204/7
- S1: value (none) -> PWR
Connections:
- removed net BTN: IC1.PB2, JP1.2, R3.1, SV2.3
- removed net LED: IC1.PB1, JP2.1, SV2.1
- removed net PWR: IC1.PB0, Q1.G, R4.1, SV2.4
- removed net READY: IC1.PB3, R2.1, SV1.16
- removed net SHUTDOWN: IC1.PB4, SV1.18
- new net ICSP-VCC: ICSP.2, VCC.1
- new net N$1: LED1.A, R2.2
- new net N$3: Q1.C, RPI.2
- new net N$4: Q1.B, R5.2, R6.1
- new net N$5: R3.2, T1.B
- new net N$6: R5.1, T1.C
- new net RPI-IO: IC2.PB3, RPI.18
- new net RPI-LED: IC2.PB2, ICSP.3, R2.1
- new net RPI-USR: IC2.PB0, ICSP.4, S1.P, S1.P1
- net +3V3: now also C3.1, IC1.OUT, IC2.VCC, VCC.2; no longer C1.1, IC1.VCC, IC2.OUT@1, JP1.1, SV2.2
- net +5V: now also C1.1, IC1.IN, J1.1, Q1.E, R6.2; no longer IC2.IN, J1.3, Q1.S, X1-1.KL
- net GND: now also C3.2, IC1.ADJ, IC2.GND, ICSP.6, J1.2, J1.3, LED1.C, RESET-B.P, RESET-B.P1, RPI.14, RPI.20, RPI.25, RPI.6, RPI.9, S1.S, S1.S1, T1.E; no longer IC1.GND, IC2.GND/ADJ, J1.1, JP2.2, R2.2, R3.2, R4.2, S1.P, S1.P1, SV1.14, SV1.20, SV1.25, SV1.6, SV1.9, SV2.6, X1-2.KL
- net RESET: now also IC2.PB5, ICSP.5, RESET-B.S, RESET-B.S1; no longer IC1.PB5, S1.S, S1.S1, SV2.5
- net RPI-PWR: now also IC2.PB1, ICSP.1, R3.1; no longer Q1.D, SV1.2
Other:
- note added: "Guillermo A. Amaral B."
- moved on the sheet: C1, C2, S1

Commit message: Updated to R2
Parts:
- removed LED1: STATUS, led:LED3MM
- removed VCC: (no value), jumper:SJ
- added PWR: (no value), gamaral:SJ-BRIDGED
- added PWR-LED: STATUS, led:LED5MM
- C2: device resistor:C-US050-024X044 -> resistor:CPOL-USE2,5-6E
Connections:
- net RPI-IO renamed RPI-IN
- new net RPI-OUT: IC2.PB4, RPI.16
- net +3V3: now also C2.+, PWR.2; no longer C2.1, VCC.2
- net GND: now also C2.-, PWR-LED.C; no longer C2.2, LED1.C
- net ICSP-VCC: now also PWR.1; no longer VCC.1
- net N$1: now also PWR-LED.A; no longer LED1.A
Changed lines of the file:
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@@
 <grid distance="0.1" unitdist="inch" unit="inch" style="lines" multiple="1" display="no" altdistance="0.01" altunitdist="inch" altunit="inch"/>
 <layers>
-<layer number="1" name="Top" color="4" fill="1" visible="no" active="no"/>
-<layer number="16" name="Bottom" color="1" fill="1" visible="no" active="no"/>
-<layer number="17" name="Pads" color="2" fill="1" visible="no" active="no"/>
-<layer number="18" name="Vias" color="2" fill="1" visible="no" active="no"/>
-<layer number="19" name="Unrouted" color="6" fill="1" visible="no" active="no"/>
-<layer number="20" name="Dimension" color="15" fill="1" visible="no" active="no"/>
-<layer number="21" name="tPlace" color="7" fill="1" visible="no" active="no"/>
-<layer number="22" name="bPlace" color="7" fill="1" visible="no" active="no"/>
-<layer number="23" name="tOrigins" color="15" fill="1" visible="no" active="no"/>
-<layer number="24" name="bOrigins" color="15" fill="1" visible="no" active="no"/>
-<layer number="25" name="tNames" color="7" fill="1" visible="no" active="no"/>
-<layer number="26" name="bNames" color="7" fill="1" visible="no" active="no"/>
-<layer number="27" name="tValues" color="7" fill="1" visible="no" active="no"/>
-<layer number="28" name="bValues" color="7" fill="1" visible="no" active="no"/>
+<layer number="1" name="Top" color="4" fill="1" visible="yes" active="no"/>
+<layer number="16" name="Bottom" color="1" fill="1" visible="yes" active="no"/>
+<layer number="17" name="Pads" color="2" fill="1" visible="yes" active="no"/>
+<layer number="18" name="Vias" color="2" fill="1" visible="yes" active="no"/>
+<layer number="19" name="Unrouted" color="6" fill="1" visible="yes" active="no"/>
+<layer number="20" name="Dimension" color="15" fill="1" visible="yes" active="no"/>
+<layer number="21" name="tPlace" color="7" fill="1" visible="yes" active="no"/>
+<layer number="22" name="bPlace" color="7" fill="1" visible="yes" active="no"/>
+<layer number="23" name="tOrigins" color="15" fill="1" visible="yes" active="no"/>
+<layer number="24" name="bOrigins" color="15" fill="1" visible="yes" active="no"/>
+<layer number="25" name="tNames" color="7" fill="1" visible="yes" active="no"/>
+<layer number="26" name="bNames" color="7" fill="1" visible="yes" active="no"/>
+<layer number="27" name="tValues" color="7" fill="1" visible="yes" active="no"/>
+<layer number="28" name="bValues" color="7" fill="1" visible="yes" active="no"/>
 <layer number="29" name="tStop" color="7" fill="3" visible="no" active="no"/>
 <layer number="30" name="bStop" color="7" fill="6" visible="no" active="no"/>
@@
 <layer number="35" name="tGlue" color="7" fill="4" visible="no" active="no"/>
 <layer number="36" name="bGlue" color="7" fill="5" visible="no" active="no"/>
-<layer number="37" name="tTest" color="7" fill="1" visible="no" active="no"/>
-<layer number="38" name="bTest" color="7" fill="1" visible="no" active="no"/>
+<layer number="37" name="tTest" color="7" fill="1" visible="yes" active="no"/>
+<layer number="38" name="bTest" color="7" fill="1" visible="yes" active="no"/>
 <layer number="39" name="tKeepout" color="4" fill="11" visible="no" active="no"/>
 <layer number="40" name="bKeepout" color="1" fill="11" visible="no" active="no"/>
@@
 <layer number="44" name="Drills" color="7" fill="1" visible="no" active="no"/>
 <layer number="45" name="Holes" color="7" fill="1" visible="no" active="no"/>
-<layer number="46" name="Milling" color="3" fill="1" visible="no" active="no"/>
-<layer number="47" name="Measures" color="7" fill="1" visible="no" active="no"/>
-<layer number="48" name="Document" color="7" fill="1" visible="no" active="no"/>
-<layer number="49" name="Reference" color="7" fill="1" visible="no" active="no"/>
-<layer number="51" name="tDocu" color="7" fill="1" visible="no" active="no"/>
-<layer number="52" name="bDocu" color="7" fill="1" visible="no" active="no"/>
+<layer number="46" name="Milling" color="3" fill="1" visible="yes" active="no"/>
+<layer number="47" name="Measures" color="7" fill="1" visible="yes" active="no"/>
+<layer number="48" name="Document" color="7" fill="1" visible="yes" active="no"/>
+<layer number="49" name="Reference" color="7" fill="1" visible="yes" active="no"/>
+<layer number="51" name="tDocu" color="7" fill="1" visible="yes" active="no"/>
+<layer number="52" name="bDocu" color="7" fill="1" visible="yes" active="no"/>
 <layer number="91" name="Nets" color="2" fill="1" visible="yes" active="yes"/>
 <layer number="92" name="Busses" color="1" fill="1" visible="yes" active="yes"/>
@@
 <part name="GND2" library="supply1" deviceset="GND" device=""/>
 <part name="C1" library="resistor" deviceset="C-US" device="050-024X044" value="100nF"/>
-<part name="C2" library="resistor" deviceset="C-US" device="050-024X044" value="10µF"/>
+<part name="C2" library="resistor" deviceset="CPOL-US" device="E2,5-6E" value="10µF"/>
 <part name="IC1" library="v-reg" deviceset="LD117A?*" device="V" technology="33"/>
 <part name="J1" library="con-jack" deviceset="DCJ0303" device=""/>
@@
 <part name="GND4" library="supply1" deviceset="GND" device=""/>
 <part name="+3V3" library="supply1" deviceset="+3V3" device=""/>
-<part name="VCC" library="jumper" deviceset="SJ" device=""/>
+<part name="PWR" library="gamaral" deviceset="SJ-BRIDGED" device=""/>
 <part name="S1" library="switch-omron" deviceset="10-XX" device="" value="PWR"/>
 <part name="RESET-B" library="switch-omron" deviceset="10-XX" device="" value="RESET"/>
 <part name="R2" library="resistor" deviceset="R-EU_" device="0204/7" value="330R"/>
-<part name="LED1" library="led" deviceset="LED" device="3MM" value="STATUS"/>
+<part name="PWR-LED" library="led" deviceset="LED" device="5MM" value="STATUS"/>
 <part name="GND5" library="supply1" deviceset="GND" device=""/>
 <part name="RPI" library="pinhead" deviceset="PINHD-2X13" device=""/>
@@
 <instance part="GND4" gate="1" x="213.36" y="91.44"/>
 <instance part="+3V3" gate="G$1" x="213.36" y="109.22"/>
-<instance part="VCC" gate="1" x="205.74" y="101.6"/>
+<instance part="PWR" gate="SJ$1" x="205.74" y="101.6"/>
 <instance part="S1" gate="1" x="124.46" y="144.78" rot="R270"/>
 <instance part="RESET-B" gate="1" x="55.88" y="132.08" rot="R270"/>
 <instance part="R2" gate="G$1" x="190.5" y="73.66"/>
-<instance part="LED1" gate="G$1" x="205.74" y="73.66" rot="R90"/>
+<instance part="PWR-LED" gate="G$1" x="205.74" y="73.66" rot="R90"/>
 <instance part="GND5" gate="1" x="213.36" y="66.04"/>
 <instance part="RPI" gate="A" x="83.82" y="50.8"/>
@@
 <wire x1="187.96" y1="134.62" x2="187.96" y2="132.08" width="0.1524" layer="91"/>
 <junction x="187.96" y="132.08"/>
-<pinref part="C2" gate="G$1" pin="2"/>
+<pinref part="C2" gate="G$1" pin="-"/>
 <wire x1="208.28" y1="134.62" x2="208.28" y2="132.08" width="0.1524" layer="91"/>
 <wire x1="208.28" y1="132.08" x2="198.12" y2="132.08" width="0.1524" layer="91"/>
@@
 </segment>
 <segment>
-<pinref part="LED1" gate="G$1" pin="C"/>
+<pinref part="PWR-LED" gate="G$1" pin="C"/>
 <pinref part="GND5" gate="1" pin="GND"/>
 <wire x1="210.82" y1="73.66" x2="213.36" y2="73.66" width="0.1524" layer="91"/>
@@
 <net name="+3V3" class="0">
 <segment>
-<pinref part="C2" gate="G$1" pin="1"/>
+<pinref part="C2" gate="G$1" pin="+"/>
 <pinref part="IC1" gate="G$1" pin="OUT"/>
 <wire x1="208.28" y1="142.24" x2="208.28" y2="144.78" width="0.1524" layer="91"/>
@@
 <pinref part="+3V3" gate="G$1" pin="+3V3"/>
 <wire x1="213.36" y1="101.6" x2="213.36" y2="106.68" width="0.1524" layer="91"/>
-<pinref part="VCC" gate="1" pin="2"/>
-<wire x1="210.82" y1="101.6" x2="213.36" y2="101.6" width="0.1524" layer="91"/>
+<pinref part="PWR" gate="SJ$1" pin="2"/>
+<wire x1="207.01" y1="101.6" x2="213.36" y2="101.6" width="0.1524" layer="91"/>
 </segment>
 </net>
@@
 </segment>
 </net>
-<net name="RPI-IO" class="0">
-<segment>
-<pinref part="IC2" gate="G$1" pin="PB3"/>
-<wire x1="101.6" y1="152.4" x2="114.3" y2="152.4" width="0.1524" layer="91"/>
-<label x="114.3" y="152.4" size="1.778" layer="95" rot="R180"/>
-</segment>
-<segment>
-<pinref part="RPI" gate="A" pin="18"/>
-<wire x1="88.9" y1="45.72" x2="104.14" y2="45.72" width="0.1524" layer="91"/>
-<label x="104.14" y="45.72" size="1.778" layer="95" rot="R180"/>
-</segment>
-</net>
 <net name="ICSP-VCC" class="0">
 <segment>
 <pinref part="ICSP" gate="A" pin="2"/>
-<pinref part="VCC" gate="1" pin="1"/>
-<wire x1="195.58" y1="101.6" x2="200.66" y2="101.6" width="0.1524" layer="91"/>
+<pinref part="PWR" gate="SJ$1" pin="1"/>
+<wire x1="195.58" y1="101.6" x2="204.47" y2="101.6" width="0.1524" layer="91"/>
 </segment>
 </net>
@@
 <segment>
 <pinref part="R2" gate="G$1" pin="2"/>
-<pinref part="LED1" gate="G$1" pin="A"/>
+<pinref part="PWR-LED" gate="G$1" pin="A"/>
 <wire x1="203.2" y1="73.66" x2="195.58" y2="73.66" width="0.1524" layer="91"/>
 </segment>
@@
 </segment>
 </net>
+<net name="RPI-OUT" class="0">
+<segment>
+<pinref part="IC2" gate="G$1" pin="PB4"/>
+<wire x1="101.6" y1="154.94" x2="114.3" y2="154.94" width="0.1524" layer="91"/>
+<label x="114.3" y="154.94" size="1.778" layer="95" rot="R180"/>
+</segment>
+<segment>
+<pinref part="RPI" gate="A" pin="16"/>
+<wire x1="88.9" y1="48.26" x2="104.14" y2="48.26" width="0.1524" layer="91"/>
+<label x="104.14" y="48.26" size="1.778" layer="95" rot="R180"/>
+</segment>
+</net>
+<net name="RPI-IN" class="0">
+<segment>
+<pinref part="IC2" gate="G$1" pin="PB3"/>
+<wire x1="101.6" y1="152.4" x2="114.3" y2="152.4" width="0.1524" layer="91"/>
+<label x="114.3" y="152.4" size="1.778" layer="95" rot="R180"/>
+</segment>
+<segment>
+<pinref part="RPI" gate="A" pin="18"/>
+<wire x1="88.9" y1="45.72" x2="104.14" y2="45.72" width="0.1524" layer="91"/>
+<label x="104.14" y="45.72" size="1.778" layer="95" rot="R180"/>
+</segment>
+</net>
